Commit message: added velocity constraint

File: turtle_brick/urdf/turtle.urdf.xacro (robot description, xacro)
@@ -3,5 +3,5 @@
     <link name="wheel">
         <visual name="wheel">
-            <origin xyz="0.0 0.0 0.0" rpy="1.570796 0.0 0.0"/>
+            <origin xyz="0.0 0.0 0.0" rpy="${pi/2} 0.0 0.0"/>
             <geometry>
                 <cylinder radius="0.5" length="0.5"/>
@@ -61,4 +61,5 @@
         <child link="wheel"/>
         <axis xyz="0.0 1.0 0.0"/>
+        <limit lower="0.0" upper="0.0" effort="0.0" velocity="${0.22/0.5}"/>
     </joint>
     <joint name="stem_base" type="continuous">

Commit message: publishing marker walls

File: turtle_brick/urdf/turtle.urdf.xacro (robot description, xacro)
@@ -1,9 +1,14 @@
 <?xml version="1.0"?>
 <robot xmlns:xacro="http://wiki.ros.org/xacro" name="brick_catcher">
+    <xacro:property name="wheel_radius" value="0.5" />
+    <xacro:property name="max_velocity" value="0.22" />
+    <xacro:property name="cyl_length" value="${wheel_radius*2}" />
+    <xacro:property name="platform_height" value ="6.0" />
+    <!-- assert that platform height must at minimum be 7*wheel_radius -->
     <link name="wheel">
         <visual name="wheel">
             <origin xyz="0.0 0.0 0.0" rpy="${pi/2} 0.0 0.0"/>
             <geometry>
-                <cylinder radius="0.5" length="0.5"/>
+                <cylinder radius="${wheel_radius}" length="${wheel_radius/2}"/>
             </geometry>
             <material name="wheel">
@@ -14,7 +19,7 @@
     <link name="stem">
         <visual name="stem">
-            <origin xyz="0.0 0.0 1.5"/>
+            <origin xyz="0.0 0.0 ${2*wheel_radius + 0.5*cyl_length}"/>
             <geometry>
-                <cylinder radius="0.5" length="1.0"/>
+                <cylinder radius="${wheel_radius}" length="${cyl_length}"/>
             </geometry>
             <material name="stem">
@@ -25,7 +30,7 @@
     <link name="base_link">
         <visual>
-            <origin xyz="0.0 0.0 2.5"/>
+            <origin xyz="0.0 0.0 ${2*wheel_radius + 1.5*cyl_length}"/>
             <geometry>
-                <box size="1.0 1.0 1.0"/>
+                <box size="${cyl_length} ${cyl_length} ${cyl_length}"/>
             </geometry>
             <material name="Cyan">
@@ -36,7 +41,7 @@
     <link name="platform_fixed">
         <visual name="fixed_cyl">
-            <origin xyz="0.0 0.0 4.0"/>
+            <origin xyz="0.0 0.0 ${2*wheel_radius + 2*cyl_length + 0.5*(platform_height-wheel_radius-2*wheel_radius-2*cyl_length)}"/>
             <geometry>
-                <cylinder radius="1.5" length="2.0"/>
+                <cylinder radius="${wheel_radius*3}" length="${platform_height-wheel_radius-2*wheel_radius-2*cyl_length}"/>
             </geometry>
             <material name="red">
@@ -47,19 +52,19 @@
     <link name="platform_tilt">
         <visual name="tilt_cyl">
-            <origin xyz="0.0 0.0 1.0"/>
+            <origin xyz="0.0 0.0 ${wheel_radius/2}"/>
             <geometry>
-                <cylinder radius="1.0" length="2.0"/>
+                <cylinder radius="${5*wheel_radius}" length="${wheel_radius}"/>
             </geometry>
             <material name="red_tilt">
-                <color rgba="0.5 0.0 0.0 1.0"/>
+                <color rgba="0.1 0.0 0.0 1.0"/>
             </material>
         </visual>
     </link>
     <joint name="wheel_stem" type="continuous">
-        <origin xyz="0.0 0.0 0.5" rpy="0.0 0.0 0.0"/>
+        <origin xyz="0.0 0.0 ${wheel_radius}" rpy="0.0 0.0 0.0"/>
         <parent link="stem"/>
         <child link="wheel"/>
         <axis xyz="0.0 1.0 0.0"/>
-        <limit lower="0.0" upper="0.0" effort="0.0" velocity="${0.22/0.5}"/>
+        <limit lower="0.0" upper="0.0" effort="0.0" velocity="${max_velocity/wheel_radius}"/>
     </joint>
     <joint name="stem_base" type="continuous">
@@ -75,5 +80,5 @@
     </joint>
     <joint name="platform_x" type="continuous">
-        <origin xyz="0.0 0.0 5.0" rpy="0.0 0.0 0.0"/>
+        <origin xyz="0.0 0.0 ${platform_height-wheel_radius}" rpy="0.0 0.0 0.0"/>
         <parent link="platform_fixed"/>
         <child link="platform_tilt"/>

Commit message: fixed rviz wall flickering

File: turtle_brick/urdf/turtle.urdf.xacro (robot description, xacro)
@@ -70,6 +70,6 @@
     <joint name="stem_base" type="continuous">
         <origin xyz="0.0 0.0 0.0" rpy="0.0 0.0 0.0"/>
-        <parent link="stem"/>
-        <child link="base_link"/>
+        <parent link="base_link"/>
+        <child link="stem"/>
         <axis xyz="0.0 0.0 1.0"/>
     </joint>

Commit message: fixed robot visuals in rviz

File: turtle_brick/urdf/turtle.urdf.xacro (robot description, xacro)
@@ -5,4 +5,6 @@
     <xacro:property name="cyl_length" value="${wheel_radius*2}" />
     <xacro:property name="platform_height" value ="6.0" />
+    <xacro:property name="base_x" value ="0.0" />
+    <xacro:property name="base_y" value ="0.0" />
     <!-- assert that platform height must at minimum be 7*wheel_radius -->
     <link name="wheel">
@@ -16,4 +18,10 @@
             </material>
         </visual>
+        <collision>
+            <origin xyz="0.0 0.0 0.0" rpy="${pi/2} 0.0 0.0"/>
+            <geometry>
+                <cylinder radius="${wheel_radius}" length="${wheel_radius/2}"/>
+            </geometry>
+        </collision>
     </link>
     <link name="stem">
@@ -27,4 +35,10 @@
             </material>
         </visual>
+        <collision>
+            <origin xyz="0.0 0.0 ${2*wheel_radius + 0.5*cyl_length}"/>
+            <geometry>
+                <cylinder radius="${wheel_radius}" length="${cyl_length}"/>
+            </geometry>
+        </collision>
     </link>
     <link name="base_link">
@@ -38,4 +52,9 @@
             </material>
         </visual>
+        <collision>
+            <geometry>
+                <box size="${cyl_length} ${cyl_length} ${cyl_length}"/>
+            </geometry>
+        </collision>
     </link>
     <link name="platform_fixed">
@@ -49,4 +68,10 @@
             </material>
         </visual>
+        <collision>
+            <origin xyz="0.0 0.0 ${2*wheel_radius + 2*cyl_length + 0.5*(platform_height-wheel_radius-2*wheel_radius-2*cyl_length)}"/>
+            <geometry>
+                <cylinder radius="${wheel_radius*3}" length="${platform_height-wheel_radius-2*wheel_radius-2*cyl_length}"/>
+            </geometry>
+        </collision>
     </link>
     <link name="platform_tilt">
@@ -60,4 +85,10 @@
             </material>
         </visual>
+        <collision>
+            <origin xyz="0.0 0.0 ${wheel_radius/2}"/>
+            <geometry>
+                <cylinder radius="${5*wheel_radius}" length="${wheel_radius}"/>
+            </geometry>
+        </collision>
     </link>
     <joint name="wheel_stem" type="continuous">

Commit message: parameters loaded from config

File: turtle_brick/urdf/turtle.urdf.xacro (robot description, xacro)
@@ -1,8 +1,12 @@
 <?xml version="1.0"?>
 <robot xmlns:xacro="http://wiki.ros.org/xacro" name="brick_catcher">
-    <xacro:property name="wheel_radius" value="0.5" />
-    <xacro:property name="max_velocity" value="0.22" />
+    <xacro:property name="yaml" value="$(find turtle_brick)/turtle.yaml" />
+    <xacro:property name="props" value="${load_yaml(yaml)}" />
+    <xacro:property name="ros_param" value="${props['/**']}" />
+    <xacro:property name="parameters" value="${ros_param['ros__parameters']}" />
+    <xacro:property name="wheel_radius" value="${parameters['wheel_radius']}" />
+    <xacro:property name="max_velocity" value="${parameters['max_velocity']}" />
     <xacro:property name="cyl_length" value="${wheel_radius*2}" />
-    <xacro:property name="platform_height" value ="6.0" />
+    <xacro:property name="platform_height" value ="${parameters['platform_height']}" />
     <xacro:property name="base_x" value ="0.0" />
     <xacro:property name="base_y" value ="0.0" />

Commit message: brick sticks to platform

File: turtle_brick/urdf/turtle.urdf.xacro (robot description, xacro)
@@ -75,5 +75,5 @@
             <origin xyz="0.0 0.0 ${2*wheel_radius + 2*cyl_length + 0.5*(platform_height-wheel_radius-2*wheel_radius-2*cyl_length)}"/>
             <geometry>
-                <cylinder radius="${wheel_radius*3}" length="${platform_height-wheel_radius-2*wheel_radius-2*cyl_length}"/>
+                <cylinder radius="${wheel_radius}" length="${platform_height-wheel_radius-2*wheel_radius-2*cyl_length}"/>
             </geometry>
         </collision>

Commit message: fixed bug when republishing brick

File: turtle_brick/urdf/turtle.urdf.xacro (robot description, xacro)
@@ -66,5 +66,5 @@
             <origin xyz="0.0 0.0 ${2*wheel_radius + 2*cyl_length + 0.5*(platform_height-wheel_radius-2*wheel_radius-2*cyl_length)}"/>
             <geometry>
-                <cylinder radius="${wheel_radius*3}" length="${platform_height-wheel_radius-2*wheel_radius-2*cyl_length}"/>
+                <cylinder radius="${wheel_radius}" length="${platform_height-wheel_radius-2*wheel_radius-2*cyl_length}"/>
             </geometry>
             <material name="red">
